Commit message: Integration of Harpoon on Husky Success

File: urdf/husky.urdf.xacro (robot description, xacro)
@@ -43,5 +43,5 @@
       <material name="black"/>
     </visual>
-    <visual name="base_link_fixed_joint_lump__arch_visual_7">
+    <!-- <visual name="base_link_fixed_joint_lump__arch_visual_7">
       <origin xyz="0.0012 0 0.251" rpy="0 0 0"/>
       <geometry>
@@ -49,5 +49,5 @@
       </geometry>
       <material name="black"/>
-    </visual>
+    </visual> -->
     <collision name="base_link_collision">
       <origin xyz="0 0 0.12" rpy="0 0 0"/>
@@ -165,3 +165,6 @@
   </joint>
   <link name="camera_depth_optical_frame"/>
+  <!-- Include the Harpoon arm -->
+  <xacro:include filename="$(find 41068_ignition_bringup)/urdf/harpoon.urdf.xacro" />
+  <xacro:harpoon_arm parent_link="base_link"/>
 </robot>
