Commit message: Projectile in Meshes

File: urdf/harpoon.urdf.xacro (robot description, xacro)
@@ -34,13 +34,13 @@
       </inertial>
       <visual>
-        <origin xyz="0 0 0.62" rpy="0 0 1.5708"/>
+        <origin xyz="0 0 0.75" rpy="0 0 1.5708"/>
         <geometry>
-          <mesh filename="package://41068_ignition_bringup/urdf/meshes/harpoon_arm/projectile.STL"/>
+          <mesh filename="package://41068_ignition_bringup/urdf/meshes/harpoon_arm/projectile.STL" scale="0.1 0.1 0.1"/>
         </geometry>
       </visual>
       <collision>
-        <origin xyz="0 0 0.62" rpy="0 0 1.5708"/>
+        <origin xyz="0 0 0.75" rpy="0 0 1.5708"/>
         <geometry>
-          <mesh filename="package://41068_ignition_bringup/urdf/meshes/harpoon_arm/projectile.STL"/>
+          <mesh filename="package://41068_ignition_bringup/urdf/meshes/harpoon_arm/projectile.STL" scale="0.1 0.1 0.1"/>
         </geometry>
       </collision>

Commit message: Harpoon Laser Script

File: urdf/harpoon.urdf.xacro (robot description, xacro)
@@ -20,4 +20,11 @@
       </visual>
     </link>
+    <!-- <gazebo reference="harpoon_barrel">
+      <plugin name="fire_projectile_plugin"
+              filename="libfire_projectile_system.so">
+        <barrel_link>harpoon_barrel</barrel_link>
+        <projectile_velocity>30.0</projectile_velocity>
+      </plugin>
+    </gazebo> -->
     <!-- Fixed joint connecting base to barrel -->
     <joint name="harpoon_joint" type="fixed">
@@ -26,5 +33,5 @@
       <origin xyz="0 0 0" rpy="0 0 0"/>
     </joint>
-    <!-- Projectile -->
+    <!-- Projectile
     <link name="harpoon_projectile">
       <inertial>
@@ -46,10 +53,10 @@
       </collision>
     </link>
-    <!-- Initially attach projectile to barrel -->
+    Initially attach projectile to barrel
     <joint name="harpoon_projectile_joint" type="fixed">
       <parent link="harpoon_barrel"/>
       <child link="harpoon_projectile"/>
       <origin xyz="0 0 0" rpy="0 0 0"/>
-    </joint>
+    </joint> -->
     <joint name="harpoon_mount" type="fixed">
       <parent link="${parent_link}"/>

File: urdf/husky.urdf.xacro (robot description, xacro)
@@ -43,5 +43,5 @@
       <material name="black"/>
     </visual>
-    <!-- <visual name="base_link_fixed_joint_lump__arch_visual_7">
+    <visual name="base_link_fixed_joint_lump__arch_visual_7">
       <origin xyz="0.0012 0 0.251" rpy="0 0 0"/>
       <geometry>
@@ -49,5 +49,5 @@
       </geometry>
       <material name="black"/>
-    </visual> -->
+    </visual>
     <collision name="base_link_collision">
       <origin xyz="0 0 0.12" rpy="0 0 0"/>

Commit message: Please work

File: urdf/harpoon.urdf.xacro (robot description, xacro)
@@ -7,5 +7,7 @@
         <origin xyz="0 0 0.25" rpy="0 0 1.5708"/>
         <geometry>
-          <mesh filename="package://41068_ignition_bringup/urdf/meshes/harpoon_arm/base.STL"/>
+          <mesh>
+            <uri>package://41068_ignition_bringup/urdf/meshes/harpoon_arm/base.STL</uri>
+          </mesh>
         </geometry>
       </visual>
@@ -16,5 +18,7 @@
         <origin xyz="0 0 0.47" rpy="0 0 1.5708"/>
         <geometry>
-          <mesh filename="package://41068_ignition_bringup/urdf/meshes/harpoon_arm/barrel.STL"/>
+          <mesh>
+            <uri>package://41068_ignition_bringup/urdf/meshes/harpoon_arm/barrel.STL</uri>
+          </mesh>
         </geometry>
       </visual>

File: urdf/husky.gazebo.xacro (robot description, xacro)
@@ -106,4 +106,29 @@
     </plugin>
   </gazebo>
+  <!-- Pose Publisher Plugin - add this after the odometry publisher plugin -->
+  <gazebo>
+    <plugin
+      filename="ignition-gazebo-pose-publisher-system"
+      name="ignition::gazebo::systems::PosePublisher">
+      <publish_link_pose>true</publish_link_pose>
+      <publish_sensor_pose>false</publish_sensor_pose>
+      <publish_collision_pose>false</publish_collision_pose>
+      <publish_visual_pose>false</publish_visual_pose>
+      <publish_nested_model_pose>false</publish_nested_model_pose>
+      <use_pose_vector_msg>true</use_pose_vector_msg>
+      <static_publisher>false</static_publisher>
+      <static_update_frequency>1</static_update_frequency>
+    </plugin>
+  </gazebo>
+  <gazebo>
+    <plugin
+      filename="ignition-gazebo-pose-publisher-system"
+      name="ignition::gazebo::systems::PosePublisher">
+      <publish_link_pose>false</publish_link_pose>
+      <publish_model_pose>true</publish_model_pose>
+      <publish_nested_model_pose>false</publish_nested_model_pose>
+      <update_frequency>10</update_frequency>
+    </plugin>
+  </gazebo>
   <gazebo reference="base_scan">
     <material>Gazebo/FlatBlack</material>
